File: pcb/moustika/_autosave-moustika.kicad_sch (KiCad schematic)
At the start: 16 parts, among them J1 Conn_01x03_Socket, J2 Conn_01x03_Socket, J3 Conn_01x03_Socket, J4 Conn_01x01_Socket, J5 Conn_01x01_Socket, J6 Conn_01x11_Pin, U1 ROB-14450, U2 QTR-8A, U4 SSD1308, U5 mini360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

Commit message: final pcb
Connections:
- net +3.3V: no longer J6.1 (Pin_1), J6.10 (Pin_10), U3.23 (3V3)
- new net: J6.1 (Pin_1), J6.10 (Pin_10), U3.23 (3V3)
Changed lines of the file:
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@@
 	)
 	(junction
-		(at 196.85 119.38)
+		(at 165.1 139.7)
 		(diameter 0)
 		(color 0 0 0 0)
 	)
 	(junction
-		(at 165.1 139.7)
+		(at 297.18 193.04)
 		(diameter 0)
 		(color 0 0 0 0)
 	)
 	(junction
-		(at 297.18 193.04)
+		(at 207.01 118.11)
 		(diameter 0)
 		(color 0 0 0 0)
@@
 	(wire
 		(pts
+			(xy 229.87 113.03) (xy 229.87 118.11)
+		)
+		(stroke
+			(width 0)
+			(type default)
+		)
+	)
+	(wire
+		(pts
 			(xy 209.55 113.03) (xy 209.55 123.19)
 		)
@@
 	(wire
 		(pts
+			(xy 207.01 118.11) (xy 207.01 113.03)
+		)
+		(stroke
+			(width 0)
+			(type default)
+		)
+	)
+	(wire
+		(pts
 			(xy 224.79 162.56) (xy 224.79 157.48)
 		)
@@
 	(wire
 		(pts
-			(xy 229.87 113.03) (xy 229.87 115.57)
-		)
-		(stroke
-			(width 0)
-			(type default)
-		)
-	)
-	(wire
-		(pts
 			(xy 165.1 123.19) (xy 165.1 124.46)
 		)
@@
 	(wire
 		(pts
-			(xy 229.87 115.57) (xy 246.38 115.57)
-		)
-		(stroke
-			(width 0)
-			(type default)
-		)
-	)
-	(wire
-		(pts
 			(xy 240.03 160.02) (xy 240.03 157.48)
 		)
@@
 	(wire
 		(pts
-			(xy 187.96 115.57) (xy 196.85 115.57)
-		)
-		(stroke
-			(width 0)
-			(type default)
-		)
-	)
-	(wire
-		(pts
 			(xy 213.36 170.18) (xy 213.36 158.75)
 		)
@@
 	(wire
 		(pts
-			(xy 207.01 119.38) (xy 207.01 113.03)
+			(xy 207.01 119.38) (xy 207.01 118.11)
 		)
 		(stroke
@@
 	(wire
 		(pts
-			(xy 196.85 115.57) (xy 196.85 119.38)
-		)
-		(stroke
-			(width 0)
-			(type default)
-		)
-	)
-	(wire
-		(pts
 			(xy 180.34 182.88) (xy 179.07 182.88)
 		)
@@
 	(wire
 		(pts
-			(xy 246.38 115.57) (xy 246.38 116.84)
+			(xy 229.87 118.11) (xy 207.01 118.11)
 		)
 		(stroke
@@
 	)
 	(symbol
-		(lib_id "power:+3.3V")
-		(at 187.96 115.57 180)
-		(unit 1)
-		(exclude_from_sim no)
-		(in_bom yes)
-		(on_board yes)
-		(dnp no)
-		(fields_autoplaced yes)
-		(property "Reference" "#PWR018"
-			(at 187.96 111.76 0)
-			(effects
-				(font
-					(size 1.27 1.27)
-				)
-				(hide yes)
-			)
-		)
-		(property "Value" "+3.3V"
-			(at 187.96 120.65 0)
-			(effects
-				(font
-					(size 1.27 1.27)
-				)
-			)
-		)
-		(property "Footprint" ""
-			(at 187.96 115.57 0)
-			(effects
-				(font
-					(size 1.27 1.27)
-				)
-				(hide yes)
-			)
-		)
-		(property "Datasheet" ""
-			(at 187.96 115.57 0)
-			(effects
-				(font
-					(size 1.27 1.27)
-				)
-				(hide yes)
-			)
-		)
-		(property "Description" "Power symbol creates a global label with name \"+3.3V\""
-			(at 187.96 115.57 0)
-			(effects
-				(font
-					(size 1.27 1.27)
-				)
-				(hide yes)
-			)
-		)
-		(pin "1"
-		)
-		(instances
-			(project "moustika"
-				(path "/7341a097-9ae3-4422-93dd-2d2a3cde0d26"
-					(reference "#PWR018")
-					(unit 1)
-				)
-			)
-		)
-	)
-	(symbol
 		(lib_id "power:PWR_FLAG")
 		(at 161.29 104.14 0)
@@
 					(unit 1)
 				)
-			)
-		)
-	)
-	(symbol
-		(lib_id "power:+3.3V")
-		(at 246.38 116.84 180)
-		(unit 1)
-		(exclude_from_sim no)
-		(in_bom yes)
-		(on_board yes)
-		(dnp no)
-		(fields_autoplaced yes)
-		(property "Reference" "#PWR01"
-			(at 246.38 113.03 0)
-			(effects
-				(font
-					(size 1.27 1.27)
-				)
-				(hide yes)
-			)
-		)
-		(property "Value" "+3.3V"
-			(at 246.38 121.92 0)
-			(effects
-				(font
-					(size 1.27 1.27)
-				)
-			)
-		)
-		(property "Footprint" ""
-			(at 246.38 116.84 0)
-			(effects
-				(font
-					(size 1.27 1.27)
-				)
-				(hide yes)
-			)
-		)
-		(property "Datasheet" ""
-			(at 246.38 116.84 0)
-			(effects
-				(font
-					(size 1.27 1.27)
-				)
-				(hide yes)
-			)
-		)
-		(property "Description" "Power symbol creates a global label with name \"+3.3V\""
-			(at 246.38 116.84 0)
-			(effects
-				(font
-					(size 1.27 1.27)
-				)
-				(hide yes)
-			)
-		)
-		(pin "1"
-		)
-		(instances
-			(project "moustika"
-				(path "/7341a097-9ae3-4422-93dd-2d2a3cde0d26"
-					(reference "#PWR01")
-					(unit 1)
-				)
