File: pcb/moustika/_autosave-moustika.kicad_sch (KiCad schematic)
At the start: 17 parts, among them J1 Conn_01x03_Socket, J2 Conn_01x03_Socket, J3 Conn_01x03_Socket, J4 Conn_01x01_Socket, J5 Conn_01x01_Socket, J6 Conn_01x11_Pin, SW1 SW_SPDT, U1 ROB-14450, U2 QTR-8A, U4 SSD1308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

Commit message: pcb adjustment
Parts:
- added SW2: SW_SPDT, Connector_PinHeader_2.54mm:PinHeader_1x03_P2.54mm_Vertical, symbol Switch:SW_SPDT
Connections:
- net +3.3V: now also SW2.2 (B), SW2.3 (C)
- net +8V: no longer J3.1 (Pin_1), SW1.2 (B)
- new net +BATT: J3.1 (Pin_1), SW1.2 (B)
- no-connect marks 30 -> 31
Other:
- moved on the sheet: SW1
