File: pcb/moustika/moustika.kicad_pcb (KiCad board)
At the start: 2 copper layers, 128.8 x 155.2 mm, 9 parts, among them J1 Conn_01x02_Socket, J2 Conn_01x02_Socket, J3 Conn_01x02_Socket, U1 ROB-14450, U2 QTR-8A, U4 SSD1308, U5 mini360, U6 mini360

Commit message: testtttt
Parts:
- added J4: Conn_01x01_Socket, Connector_PinHeader_2.54mm:PinHeader_1x01_P2.54mm_Vertical, F.Cu at (274.5, 263.6)
- added J5: Conn_01x01_Socket, Connector_PinHeader_2.54mm:PinHeader_1x01_P2.54mm_Vertical, F.Cu at (255.9, 267.9)
- added J6: Conn_01x11_Pin, Connector_PinHeader_2.54mm:PinHeader_1x11_P2.54mm_Vertical, F.Cu at (282.6, 226.8)
- added S1: BUTT-2, spo2_stuff:SW_BUTT-2, F.Cu at (221.6, 234.1)
- added S2: BUTT-2, spo2_stuff:SW_BUTT-2, F.Cu at (212.4, 242.6)
- added S3: BUTT-2, spo2_stuff:SW_BUTT-2, F.Cu at (221.6, 249.2)
- added S4: BUTT-2, spo2_stuff:SW_BUTT-2, F.Cu at (230.7, 242.5)
- J1, J2, J3: value Conn_01x02_Socket -> Conn_01x03_Socket; footprint Connector_PinHeader_1.00mm:PinHeader_1x02_P1.00mm_Vertical -> Connector_PinHeader_2.54mm:PinHeader_1x03_P2.54mm_Vertical
- moved U6 280.3 mm to (308.8, 277.5)
- moved U4 221.4 mm to (318.0, 249.5), turned to 0 degrees
- moved U3 217.2 mm to (295.1, 260.1)
- moved U1 213.4 mm to (268.0, 280.6)
- moved J1 209.5 mm to (323.4, 284.3)
- moved U2 208.7 mm to (289.4, 133.8)
- moved J3 206.1 mm to (222.6, 215.6)
- moved J2 204.5 mm to (218.6, 284.3)
- moved U5 162.4 mm to (239.6, 277.5)
Connections:
- J1 pad 2: Net-(J1-Pin_2) -> unconnected-(J1-Pin_2-Pad2)
- J2 pad 2: Net-(J2-Pin_2) -> unconnected-(J2-Pin_2-Pad2)
- J3 pad 2: GND -> unconnected-(J3-Pin_2-Pad2)
- U1 pad 16: Net-(U1-PWMA) -> Net-(J5-Pin_1)
- U1 pad 5: Net-(J2-Pin_2) -> Net-(J2-Pin_3)
- U1 pad 6: Net-(J1-Pin_2) -> Net-(J1-Pin_3)
- U2 pad 3V3: +3.3V -> unconnected-(U2-Pad3V3)
- U2 pad GND: Net-(U2-PadGND) -> unconnected-(U2-PadGND)
- U2 pad LED1: Net-(U3-A7) -> unconnected-(U2-PadLED1)
- U2 pad LED2: Net-(U3-A6) -> unconnected-(U2-PadLED2)
- U2 pad LED3: Net-(U3-A5) -> unconnected-(U2-PadLED3)
- U2 pad LED4: Net-(U3-A4) -> unconnected-(U2-PadLED4)
- U2 pad LED5: Net-(U3-A3) -> unconnected-(U2-PadLED5)
- U2 pad LED6: Net-(U3-A2) -> unconnected-(U2-PadLED6)
- U2 pad LED7: Net-(U3-A1) -> unconnected-(U2-PadLED7)
- U2 pad LED8: Net-(U3-A0) -> unconnected-(U2-PadLED8)
- U2 pad LED_ON: Net-(U2-PadLED_ON) -> unconnected-(U2-PadLED_ON)
- U3 pad 12: Net-(U1-PWMA) -> Net-(J4-Pin_1)
- U3 pad 19: unconnected-(U3-GND-Pad19) -> GND
- U3 pad 20: unconnected-(U3-3V3-Pad20) -> +3.3V
- U3 pad 22: Net-(U2-PadGND) -> Net-(J6-Pin_11)
- U3 pad 23: Net-(U2-PadLED_ON) -> +3.3V
- U3 pad 28: Net-(U3-A7) -> Net-(J6-Pin_9)
- U3 pad 29: Net-(U3-A6) -> Net-(J6-Pin_8)
- U3 pad 30: Net-(U3-A5) -> Net-(J6-Pin_7)
- U3 pad 31: Net-(U3-A4) -> Net-(J6-Pin_6)
- U3 pad 32: Net-(U3-A3) -> Net-(J6-Pin_5)
- U3 pad 33: Net-(U3-A2) -> Net-(J6-Pin_4)
- U3 pad 34: Net-(U3-A1) -> Net-(J6-Pin_3)
- U3 pad 35: Net-(U3-A0) -> Net-(J6-Pin_2)
- U6 pad 1: +8V -> +3.3V
Routing:
- net +8V: track 64.4 -> 297.4 mm
- net GND: track 65.3 -> 280.0 mm
- net +3.3V: track 0.00 -> 174.4 mm
- net Net-(J1-Pin_3): track 0.00 -> 60.4 mm
- net Net-(J2-Pin_3): track 0.00 -> 60.0 mm
- net Net-(J1-Pin_2): track 56.0 -> 0.00 mm
- net Net-(J2-Pin_2): track 49.6 -> 0.00 mm
- net +5V: track 0.00 -> 49.3 mm
- net Net-(U3-B12): track 0.00 -> 44.4 mm
- net Net-(U3-B15): track 0.00 -> 40.5 mm
- net Net-(U3-B13): track 0.00 -> 27.9 mm
- net Net-(U3-B7): track 34.6 -> 60.7 mm
- net Net-(U3-B14): track 0.00 -> 24.7 mm
- net Net-(J6-Pin_11): track 0.00 -> 19.4 mm
- net Net-(J6-Pin_9): track 0.00 -> 15.2 mm
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Other:
- board size 128.8 x 155.2 mm -> 140 x 169 mm
