File: pcb/moustika/moustika.kicad_pcb (KiCad board)
At the start: 2 copper layers, 140 x 169 mm, 16 parts, among them J1 Conn_01x03_Socket, J2 Conn_01x03_Socket, J3 Conn_01x03_Socket, J4 Conn_01x01_Socket, J5 Conn_01x01_Socket, J6 Conn_01x11_Pin, U1 ROB-14450, U2 QTR-8A, U4 SSD1308, U5 mini360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

Commit message: fixed the chassis
Parts:
- moved U2 107.6 mm to (320.6, 30.8)
- moved J4 105.9 mm to (304.3, 162.0)
- moved S1 105.9 mm to (251.4, 132.4)
- moved U1 105.9 mm to (297.8, 179.0)
- moved J6 105.9 mm to (312.4, 125.2)
- moved J1 105.9 mm to (353.2, 182.7)
- moved J2 105.9 mm to (248.4, 182.7)
- moved J3 105.9 mm to (252.4, 114.0)
- moved S3 105.9 mm to (251.4, 147.6)
- moved S4 105.9 mm to (260.5, 140.9)
- moved U4 105.9 mm to (347.8, 147.9)
- moved U5 105.9 mm to (269.4, 175.9)
- moved U6 105.9 mm to (338.6, 175.9)
- moved S2 105.9 mm to (242.2, 141.0)
- moved J5 105.9 mm to (285.7, 166.3)
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Other:
- outline, holes or cut-outs redrawn
